File: hardware/Jacquard_Machine_Brain/Jacquard_Machine_Brain.kicad_sch (KiCad schematic)
At the start: 38 parts, among them J1 Terminal Block, J13 Molex Micro-Fit 4pos, J15 USB_A, J16 Wurth_RJ45_LED, SW1 SW_DIP_x02, SW2 SW_MEC_5G, U1 R-78E5.0-1.0, U2 Teensy4.1, U6 AO4882

Commit message: Further progress on the brain
Parts:
- added C10, C11, C12, C6, C7, C8, C9: 0.1uF, Capacitor_SMD:C_0402_1005Metric, symbol Device:C_Small
- added J2: Conn_01x08, Connector_PinSocket_2.54mm:PinSocket_1x08_P2.54mm_Vertical, symbol Connector_Generic:Conn_01x08
- added J3: JST-SH 01x04, Connector_JST:JST_SH_BM04B-SRSS-TB_1x04-1MP_P1.00mm_Vertical, symbol Connector_Generic:Conn_01x04
- added J4, J5: Conn_01x02, Connector_PinSocket_2.54mm:PinSocket_1x02_P2.54mm_Vertical, symbol Connector_Generic:Conn_01x02
- added JP1, JP2, JP5, JP6: SolderJumper_2_Bridged, Jumper:SolderJumper-2_P1.3mm_Bridged_RoundedPad1.0x1.5mm, symbol Jumper:SolderJumper_2_Bridged
- added JP3, JP4: SolderJumper_3_Bridged12, Jumper:SolderJumper-3_P1.3mm_Bridged12_RoundedPad1.0x1.5mm_NumberLabels, symbol Jumper:SolderJumper_3_Bridged12
- added R10: 200k, Resistor_SMD:R_0402_1005Metric, symbol Device:R_Small
- added R11, R14, R2: 100, Resistor_SMD:R_0402_1005Metric, symbol Device:R_Small
- added R15, R16: 4.7k, Resistor_SMD:R_0603_1608Metric, symbol Device:R_Small
- added R76: 0Ω, Resistor_SMD:R_0805_2012Metric, symbol Device:R_Small
- added U10, U3, U4, U7, U8: 74AHCT1G125, Package_TO_SOT_SMD:SOT-353_SC-70-5, symbol 0_integrated_circuits:74AHCT1G125
- added U5: 74AHCT125, Package_SO:TSSOP-14_4.4x5mm_P0.65mm, symbol 0_integrated_circuits:74AHCT125_Multi
- added U9: PCA9306D, Package_SO:SO-8_3.9x4.9mm_P1.27mm, symbol Interface:PCA9306D
- J13: value Molex Micro-Fit 4pos -> ~; footprint 0_connector:MOLEX_MICROFIT-RA-4POS_436500400 -> Connector_PinSocket_2.54mm:PinSocket_1x04_P2.54mm_Vertical; Link https://www.digikey.com/en/products/detail/molex/0436500400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 -> (none); Manu # 0436500400 -> (none); Manu. MOLEX -> (none)
- R12, R13: value 10k -> 4.7k; footprint Resistor_SMD:R_0805_2012Metric_Pad1.20x1.40mm_HandSolder -> Resistor_SMD:R_0603_1608Metric; LCSC (none) -> C23162; Link https://mou.sr/4vBd3uS -> (none); Manu # RE0805FRE1010KL -> 0603WAF4701T5E; Manu. YAGEO -> UNI-ROYAL(Uniroyal Elec); Package 0805 -> 0603
Connections:
- net LED_GND is gone; now on net GND: D3.1 (K), D4.1 (K)
- net +12V: now also J4.1 (Pin_1), J5.1 (Pin_1)
- net +3V3: now also U2.46 (3V3), U9.2 (VREF1)
- net +5V: now also C10.1, C11.1, C12.1, C6.1, C7.1, C8.1, J2.2 (Pin_2), R10.1, R15.1, R16.1, U10.5 (VCC), U3.5 (VCC), U4.5 (VCC), U7.5 (VCC), U8.5 (VCC)
- net BUTTON_0: now also J2.5 (Pin_5)
- net GATE_1: now also U3.4 (Y); no longer R4.1
- net GATE_2: now also U8.4 (Y); no longer R5.1
- net GND: now also C10.2, C11.2, C12.2, C6.2, C7.2, C8.2, C9.2, J2.1 (Pin_1), J3.1 (Pin_1), R76.1, U10.1 (~{OE}), U10.3 (GND), U3.1 (~{OE}), U3.3 (GND), U4.1 (~{OE}), U4.3 (GND), U7.1 (~{OE}), U7.3 (GND), U8.1 (~{OE}), U8.3 (GND), U9.1 (GND)
- net GNDPWR: now also R76.2
- net SCL_0: now also J2.4 (Pin_4), JP3.2 (C); no longer J13.4 (Pin_4), JP8.1 (A), U2.41 (19_A5_SCL)
- net SDA_0: now also J2.3 (Pin_3), JP4.2 (C); no longer J13.3 (Pin_3), JP7.1 (A), U2.40 (18_A4_SDA)
- net DRAIN_1: no longer names the net of D5.2 (A), U6.7 (D), U6.8 (D)
- net DRAIN_1: now also J5.2 (Pin_2)
- net DRAIN_2: no longer names the net of D6.2 (A), U6.5 (D), U6.6 (D)
- net DRAIN_2: now also J4.2 (Pin_2)
- new net: JP6.2 (B), R16.2
- new net: JP5.2 (B), R15.2
- new net: C9.1, R10.2, U9.7 (VREF2), U9.8 (EN)
- new net: J3.3 (Pin_3), R14.1
- new net: J3.2 (Pin_2), R11.1
- new net: J3.4 (Pin_4), R2.1
- new net BUTTON_1: J2.6 (Pin_6)
- new net BUTTON_2: J2.7 (Pin_7)
- new net BUTTON_3: J2.8 (Pin_8)
- new net LATCH_3.3V: U7.2 (A)
- new net LATCH_5V: R14.2, U7.4 (Y)
- new net MOSFET_1: U3.2 (A)
- new net MOSFET_2: U8.2 (A)
- new net SCL_0_3.3V: JP3.3 (B), JP7.1 (A), U2.41 (19_A5_SCL), U9.3 (SCL1)
- new net SCL_0_5V: JP3.1 (A), JP5.1 (A), U9.6 (SCL2)
- new net SCL_1: J13.4 (Pin_4), JP2.1 (A)
- new net SDA_0_3.3V: JP4.3 (B), JP8.1 (A), U2.40 (18_A4_SDA), U9.4 (SDA1)
- new net SDA_0_5V: JP4.1 (A), JP6.1 (A), U9.5 (SDA2)
- new net SDA_1: J13.3 (Pin_3), JP1.1 (A)
- new net SERIAL_DATA_3.3V: U10.2 (A)
- new net SERIAL_DATA_5V: R2.2, U10.4 (Y)
- new net SRCLK_3.3V: U4.2 (A)
- new net SRCLK_5V: R11.2, U4.4 (Y)
Other:
- note added: "POWER GROUND TO DIGITAL GROUND TIE POINT"
- moved on the sheet: D3, D4, D5, D6, J13, JP7, JP8, R12, R4, R5, R6, R7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
