File: hardware/Jacquard_Machine_Brain/Jacquard_Machine_Brain.kicad_pcb (KiCad board)
At the start: 2 copper layers, 160 x 70 mm, 69 parts, among them J1 Terminal Block, J15 USB_A, J16 Wurth_RJ45_LED, J2 Conn_01x08, J3 JST-SH 01x04, J4 Conn_01x02, J5 Conn_01x02, SW1 SW_DIP_x02, SW2 SW_MEC_5G, U1 R-78E5.0-1.0, U10 74AHCT1G125, U2 Teensy4.1, U3 74AHCT1G125, U4 74AHCT1G125, U5 74AHCT125, U6 AO4882, U7 74AHCT1G125, U8 74AHCT1G125, U9 PCA9306D

Commit message: sync
Parts:
- moved C10 156.5 mm to (170.2, -3.50)
- moved C11 156.5 mm to (170.2, -1.53)
- moved C12 156.5 mm to (170.2, 0.44)
- moved C6 156.5 mm to (170.2, -11.4)
- moved C7 156.5 mm to (170.2, -9.41)
- moved C8 156.5 mm to (170.2, -7.44)
- moved C9 156.5 mm to (170.2, -5.47)
- moved D3 156.5 mm to (185.5, 2.42)
- moved D4 156.5 mm to (185.5, 4.41)
- moved D5 156.5 mm to (171.7, 13.1)
- moved D6 156.5 mm to (171.7, 16.4)
- moved J13 156.5 mm to (182.4, -10.0)
- moved J2 156.5 mm to (157.9, -10.0)
- moved J4 156.5 mm to (176.9, 3.75)
- moved J5 156.5 mm to (181.5, 3.75)
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Other:
- outline, holes or cut-outs redrawn

Commit message: Progress check
Parts:
- removed J16: Wurth_RJ45_LED, 0_connector:Wurth_7499010211A_RJ45
- removed JP2, JP5, JP6, JP7, JP8: SolderJumper_2_Bridged, Jumper:SolderJumper-2_P1.3mm_Bridged_RoundedPad1.0x1.5mm
- removed R12, R13: 4.7k, Resistor_SMD:R_0603_1608Metric
- removed SW1: SW_DIP_x02, Button_Switch_THT:SW_DIP_SPSTx02_Slide_9.78x7.26mm_W7.62mm_P2.54mm
- removed SW2: SW_MEC_5G, Button_Switch_THT:SW_TH_Tactile_Omron_B3F-100x
- removed U5: 74AHCT125, Package_SO:TSSOP-14_4.4x5mm_P0.65mm
- added J200: WIZnet_J1B1211CCD_RJ45, 0_connector:WIZnet_J1B1211CCD_RJ45, F.Cu at (118.9, 109.2)
- added R17: 4.7k, Resistor_SMD:R_0603_1608Metric, F.Cu at (223.4, 84.0)
- added R18: 4.7k, Resistor_SMD:R_0603_1608Metric, F.Cu at (223.1, 87.5)
- added R19: 4.7k, Resistor_SMD:R_0603_1608Metric, F.Cu at (211.0, 72.2)
- added R20: 4.7k, Resistor_SMD:R_0603_1608Metric, F.Cu at (207.2, 72.2)
- C3: footprint Capacitor_SMD:C_0805_2012Metric_Pad1.18x1.45mm_HandSolder -> Capacitor_SMD:C_0805_2012Metric
- C9: value 0.1uF -> 100pF
- JP1: value SolderJumper_2_Bridged -> SolderJumper_3_Bridged123; footprint Jumper:SolderJumper-2_P1.3mm_Bridged_RoundedPad1.0x1.5mm -> Jumper:SolderJumper-3_P1.3mm_Open_RoundedPad1.0x1.5mm
- JP3, JP4: moved to B.Cu
- R3: value 330 -> 220R; footprint Resistor_SMD:R_0805_2012Metric_Pad1.20x1.40mm_HandSolder -> Resistor_SMD:R_0805_2012Metric
- moved JP1 118.5 mm to (221.8, 92.0)
- moved U4 112.6 mm to (111.2, 91.6), turned to 180 degrees
- moved C12 111.0 mm to (110.5, 94.0)
- moved C11 108.7 mm to (110.5, 89.2)
- moved J13 107.2 mm to (231.8, 85.2)
- moved C10 106.3 mm to (110.5, 84.5)
- moved U7 105.2 mm to (111.2, 86.9), turned to 180 degrees
- moved R2 104.9 mm to (103.8, 83.5)
- moved R11 103.7 mm to (103.8, 85.5)
- moved R14 101.5 mm to (103.8, 84.5)
- moved U10 94.7 mm to (111.2, 82.2), turned to 180 degrees
- moved J2 87.0 mm to (212.5, 57.8), turned to 90 degrees
- moved C6 83.6 mm to (204.3, 65.0), turned to 180 degrees
- moved U3 83.2 mm to (199.5, 66.0), turned to 90 degrees
- moved R15 82.3 mm to (222.5, 68.0), turned to 90 degrees
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Connections:
- net Net-(J1-Pin_1) renamed /PWR_IN
- C3 pad 1: Net-(C3-Pad1) -> GND
- C3 pad 2: GND -> Net-(C3-Pad2)
- C6 pad 1: +5V -> +3V3
- JP1 pad 1: SDA_1 -> Net-(JP1-A)
- JP1 pad 2: unconnected-(JP1-B-Pad2) -> +3V3
- R15 pad 2: Net-(JP5-B) -> SCL_0_5V
- R16 pad 2: Net-(JP6-B) -> SDA_0_5V
- R4 pad 1: unconnected-(R4-Pad1) -> GATE_1
- R5 pad 1: unconnected-(R5-Pad1) -> GATE_2
- U2 pad 32: unconnected-(U2-40_A16-Pad32) -> MOSFET_1
- U2 pad 33: unconnected-(U2-41_A17-Pad33) -> MOSFET_2
- U2 pad 43: unconnected-(U2-21_A7_RX5_BCLK1-Pad43) -> LATCH_3.3V
- U2 pad 44: unconnected-(U2-22_A8_CTX1-Pad44) -> SRCLK_3.3V
- U2 pad 45: unconnected-(U2-23_A9_CRX1_MCLK1-Pad45) -> SERIAL_DATA_3.3V
Routing:
- net SCL_0_3.3V: track 0.00 -> 78.5 mm, vias 0 -> 2
- net SDA_0_3.3V: track 0.00 -> 58.6 mm, vias 0 -> 2
- net LATCH_3.3V: track 0.00 -> 50.9 mm, vias 0 -> 1
- net SRCLK_3.3V: track 0.00 -> 50.3 mm
- net GNDPWR: track 27.1 -> 72.9 mm
- net SERIAL_DATA_3.3V: track 0.00 -> 43.9 mm
- net +5V: track 38.6 -> 76.3 mm, vias 0 -> 3
- net Net-(R4-Pad2): track 0.00 -> 35.9 mm
- net Net-(R5-Pad2): track 0.00 -> 31.9 mm
- net Net-(D5-A): track 0.00 -> 21.4 mm
- net Net-(U1-IN): track 15.7 -> 34.3 mm
- net MOSFET_1: track 0.00 -> 18.2 mm
- net SCL_0_5V: track 0.00 -> 17.9 mm, vias 0 -> 1
- net /PWR_IN: track 34.9 -> 17.2 mm
- net +3V3: track 0.00 -> 16.9 mm
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- added copper zone on B.Cu, net GND
- added copper zone on F.Cu, net GND
Other:
- outline, holes or cut-outs redrawn
- board text removed: "12V!"

Commit message: sync
Parts:
- removed J13: ~, Connector_PinSocket_2.54mm:PinSocket_1x04_P2.54mm_Vertical
- added J6: Conn_02x08_Odd_Even, Connector_PinSocket_2.54mm:PinSocket_2x08_P2.54mm_Vertical, F.Cu at (169.8, 107.0)
- added REF**: GVH_Cloak_Figure, 0_logo:GVH_Cloak_Figure, F.Cu at (248.5, 84.5)
- moved JP1 60.7 mm to (161.5, 98.5), turned to 90 degrees
- moved R17 57.4 mm to (167.8, 97.8)
- moved R18 56.7 mm to (167.8, 99.8)
- moved C4 14.6 mm to (151.2, 62.1)
- moved C5 1.25 mm to (142.8, 62.1)
- moved J5 0.21 mm to (173.0, 62.8)
Connections:
- U2 pad 12: unconnected-(U2-10_CS_MQSR-Pad12) -> SPI_CS
- U2 pad 13: unconnected-(U2-11_MOSI_CTX1-Pad13) -> SPI_MOSI
- U2 pad 14: NIC_LED -> SPI_MISO
- U2 pad 15: unconnected-(U2-3V3-Pad15) -> +3V3
- U2 pad 16: unconnected-(U2-24_A10_TX6_SCL2-Pad16) -> UART_TX_6
- U2 pad 17: unconnected-(U2-25_A11_RX6_SDA2-Pad17) -> UART_RX_6
- U2 pad 28: unconnected-(U2-36_CS-Pad28) -> GPIO_4
- U2 pad 29: unconnected-(U2-37_CS-Pad29) -> GPIO_3
- U2 pad 30: unconnected-(U2-38_CS1_IN1-Pad30) -> GPIO_2
- U2 pad 31: unconnected-(U2-39_MISO1_OUT1A-Pad31) -> GPIO_1
- U2 pad 35: unconnected-(U2-13_SCK_LED-Pad35) -> SPI_CLK
- U2 pad 38: unconnected-(U2-16_A2_RX4_SCL1-Pad38) -> SCL_1
- U2 pad 39: unconnected-(U2-17_A3_TX4_SDA1-Pad39) -> SDA_1
- U2 pad 4: unconnected-(U2-2_OUT2-Pad4) -> NIC_LED
- U2 pad 46: +3V3 -> unconnected-(U2-3V3-Pad46)
Routing:
- net +5V: track 76.3 -> 223.1 mm, vias 3 -> 8
- net +3V3: track 16.9 -> 98.8 mm, vias 0 -> 1
- net SPI_CLK: track 0.00 -> 36.4 mm
- net GPIO_1: track 0.00 -> 34.7 mm, vias 0 -> 1
- net GPIO_3: track 0.00 -> 34.7 mm, vias 0 -> 1
- net GPIO_2: track 0.00 -> 34.7 mm, vias 0 -> 1
- net GPIO_4: track 0.00 -> 34.7 mm, vias 0 -> 1
- net SCL_1: track 0.00 -> 33.9 mm
- net SDA_1: track 0.00 -> 32.8 mm
- net NIC_LED: track 0.00 -> 22.8 mm, vias 0 -> 1
- net UART_TX_6: track 0.00 -> 20.2 mm
- net SPI_MOSI: track 0.00 -> 20.2 mm
- net SPI_CS: track 0.00 -> 20.2 mm
- net UART_RX_6: track 0.00 -> 20.2 mm
- net SPI_MISO: track 0.00 -> 20.2 mm
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Other:
- board text added: "10"
- board text added: "11"
- board text added: "12"
- board text added: "13"
- board text added: "16"
- board text added: "17"
- board text added: "18"
- board text added: "19"
- board text added: "21"
- board text added: "22"
- board text added: "23"
- board text added: "24"
- board text added: "25"
- board text added: "3.3V"
- board text added: "36"
- board text added: "37"
- board text added: "38"
- board text added: "39"
- board text added: "40"
- board text added: "41"
- board text added: "BUT1"
- board text added: "BUT2"
- board text added: "BUT3"
- board text added: "BUT4"
- board text added: "CLOCK"
- board text added: "DATA"
- board text added: "FET1"
- board text added: "FET2"
- board text added: "GND"
- board text added: "J6"
- board text added: "LATCH"
- board text added: "SCL"
- board text added: "SDA"

Commit message: Connected the UI buttons
Parts:
- moved D2 18.6 mm to (151.0, 59.1)
- moved C4 7.18 mm to (144.8, 59.1)
- moved C5 7.18 mm to (136.2, 59.1)
Connections:
- U2 pad 21: unconnected-(U2-29_TX7-Pad21) -> BUTTON_0
- U2 pad 22: unconnected-(U2-30_CRX3-Pad22) -> BUTTON_1
- U2 pad 23: unconnected-(U2-31_CTX3-Pad23) -> BUTTON_2
- U2 pad 24: unconnected-(U2-32_OUT1B-Pad24) -> BUTTON_3
Routing:
- net BUTTON_0: track 0.00 -> 49.5 mm
- net BUTTON_3: track 0.00 -> 49.4 mm
- net BUTTON_1: track 0.00 -> 49.0 mm
- net BUTTON_2: track 0.00 -> 48.8 mm
- net GND: track 17.6 -> 28.2 mm, vias 55 -> 69
- net GNDPWR: track 70.7 -> 76.0 mm

Commit message: PCB Wrap up
Parts:
- moved REF** 104.0 mm to (145.8, 68.5)
Other:
- board text added: "Jacquard Machine Brain v1.0"
