File: hardware/Jacquard_Machine_Driver/Jacquard_Machine_Driver.kicad_pcb (KiCad board)
At the start: 2 copper layers, 50 x 77 mm, 165 parts, among them J1 Terminal Block, J2 JST-SH 01x04, J3 JST-SH 01x04, J4 Conn_02x08_Odd_Even, J5 Conn_02x08_Odd_Even, J6 Conn_02x08_Odd_Even, U1 R-78E5.0-1.0, U10 AO4882, U11 AO4882, U12 AO4882, U13 AO4882, U14 AO4882, U15 AO4882, U16 AO4882, U17 AO4882, U2 SN74LVC2G17, U3 74HC595, U4 74HC595, U5 74HC595, U6 AO4882, U7 AO4882, U8 AO4882, U9 AO4882

Commit message: sync
Other:
- board text removed: "Jacquard Driver PCB • V1.0 Daniel Bornhorst • 05/2026"
Changed lines of the file:
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@@
 			)
 		)
-		(property "LCSC" "-"
+		(property "LCSC" "C30734"
 			(at 0 0 270)
 			(unlocked yes)
@@
 			)
 		)
-		(property "LCSC" "-"
+		(property "LCSC" "C22371890"
 			(at 0 0 0)
 			(unlocked yes)
@@
 			)
 		)
-		(property "Link" "https://www.mouser.com/ProductDetail/Samsung-Electro-Mechanics/CL31B225KBHNNNE?qs=349EhDEZ59oNolj3jR402w%3D%3D"
+		(property "Link" "https://www.mouser.com/ProductDetail/Samsung-Electro-Mechanics/CL21A225KBQNNNE?qs=xZ%2FP%252Ba9zWqaBMj9IHA8rdw%3D%3D"
 			(at 0 0 90)
 			(unlocked yes)
@@
 			)
 		)
-		(property "Manu #" "CL31B225KBHNNNE"
+		(property "Manu #" "CL21A225KBQNNNE"
 			(at 0 0 90)
 			(unlocked yes)
@@
 			)
 		)
-		(property "LCSC" "C50254"
+		(property "LCSC" "C377773"
 			(at 0 0 90)
 			(unlocked yes)
@@
 			)
 		)
-		(property "LCSC" "-"
+		(property "LCSC" "C151075"
 			(at 0 0 180)
 			(unlocked yes)
@@
 			)
 		)
-		(property "LCSC" "-"
+		(property "LCSC" "C89123"
 			(at 0 0 0)
 			(unlocked yes)
@@
 			)
 		)
-		(property "LCSC" "-"
+		(property "LCSC" "C30734"
 			(at 0 0 270)
 			(unlocked yes)
@@
 			)
 		)
-		(property "LCSC" "-"
+		(property "LCSC" "C30734"
 			(at 0 0 270)
 			(unlocked yes)
@@
 		)
 	)
-	(gr_text "Jacquard Driver PCB • V1.0\nDaniel Bornhorst • 05/2026"
-		(at 124.5 167 -0)
-		(layer "B.SilkS")
-		(effects
-			(font
-				(size 1.27 1.27)
-				(thickness 0.2032)
-			)
-			(justify mirror)
-		)
-	)
 	(dimension
 		(type orthogonal)
@@
 			(thermal_bridge_width 0.5)
 			(smoothing fillet)
-			(radius 10)
+			(radius 2)
 		)
 		(polygon
