File: hardware/Jacquard_Machine_Driver/Jacquard_Machine_Driver.kicad_sch (KiCad schematic)
At the start: 32 parts, among them J1 Terminal Block, J2 JST-SH 01x04, J3 JST-SH 01x04, J4 Conn_02x08_Odd_Even, J5 Conn_02x08_Odd_Even, J6 Conn_02x08_Odd_Even, U1 R-78E5.0-1.0, U2 SN74LVC2G17, U3 74HC595, U4 74HC595, U5 74HC595

Commit message: sync
Parts:
- C2: LCSC C50254 -> C377773; Link https://www.mouser.com/ProductDetail/Samsung-Electro-Mechanics/CL31B225KBHNNNE?qs=349EhDEZ59oNolj3jR402w%3D%3D -> https://www.mouser.com/ProductDetail/Samsung-Electro-Mechanics/CL21A225KBQNNNE?qs=xZ%2FP%252Ba9zWqaBMj9IHA8rdw%3D%3D; Manu # CL31B225KBHNNNE -> CL21A225KBQNNNE
- F1: LCSC - -> C151075
- J1: LCSC - -> C89123
- J4, J5, J6: LCSC - -> C30734
- R2, R3: Manu # 0402WGF1000TCE -> 0402WGF1000TCE
- U1: LCSC - -> C22371890
Connections:
- net SRCLK_IN: now reaches J2.2 (Pin_2), U2.1 (1A)
- net LATCH_IN: now reaches J2.3 (Pin_3), U2.3 (2A)
Other:
- note added: "IN"
- note added: "OUT"
- moved on the sheet: C3
Changed lines of the file:
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@@
 		)
 	)
+	(text "OUT"
+		(exclude_from_sim no)
+		(at 109.22 154.178 0)
+		(effects
+			(font
+				(size 1.905 1.905)
+			)
+		)
+	)
 	(text "INDICATOR LEDs\nDISCONNECT\nJUMPER"
 		(exclude_from_sim no)
@@
 		)
 	)
+	(text "IN"
+		(exclude_from_sim no)
+		(at 25.654 154.178 0)
+		(effects
+			(font
+				(size 1.905 1.905)
+			)
+		)
+	)
 	(text "12V INPUT"
 		(exclude_from_sim no)
@@
 		)
 	)
+	(label "SRCLK_IN"
+		(at 40.64 161.29 0)
+		(effects
+			(font
+				(size 1.27 1.27)
+			)
+			(justify left bottom)
+		)
+	)
 	(label "SOLENOID_18"
 		(at 336.55 166.37 180)
@@
 		)
 	)
+	(label "LATCH_IN"
+		(at 40.64 163.83 0)
+		(effects
+			(font
+				(size 1.27 1.27)
+			)
+			(justify left bottom)
+		)
+	)
 	(label "SOLENOID_9"
 		(at 271.78 91.44 0)
@@
 	(symbol
 		(lib_id "power:GND")
-		(at 114.3 149.86 0)
+		(at 120.65 149.86 0)
 		(unit 1)
 		(exclude_from_sim no)
@@
 		(dnp no)
 		(property "Reference" "#PWR06"
-			(at 114.3 156.21 0)
+			(at 120.65 156.21 0)
 			(effects
 				(font
@@
 		)
 		(property "Value" "GND"
-			(at 114.427 154.2542 0)
+			(at 120.777 154.2542 0)
 			(effects
 				(font
@@
 		)
 		(property "Footprint" ""
-			(at 114.3 149.86 0)
+			(at 120.65 149.86 0)
 			(effects
 				(font
@@
 		)
 		(property "Datasheet" ""
-			(at 114.3 149.86 0)
+			(at 120.65 149.86 0)
 			(effects
 				(font
@@
 		)
 		(property "Description" ""
-			(at 114.3 149.86 0)
+			(at 120.65 149.86 0)
 			(effects
 				(font
@@
 			)
 		)
-		(property "LCSC" "-"
+		(property "LCSC" "C30734"
 			(at 344.17 171.45 0)
 			(effects
@@
 			)
 		)
-		(property "Manu #" " 0402WGF1000TCE"
+		(property "Manu #" "0402WGF1000TCE"
 			(at 88.9 163.83 0)
 			(effects
@@
 			)
 		)
-		(property "Digikey P/N" ""
-			(at 88.9 163.83 90)
-			(effects
-				(font
-					(size 1.27 1.27)
-				)
-				(hide yes)
-			)
-		)
-		(property "Digikey Page" ""
-			(at 88.9 163.83 90)
-			(effects
-				(font
-					(size 1.27 1.27)
-				)
-				(hide yes)
-			)
-		)
 		(pin "2"
 		)
@@
 	(symbol
 		(lib_id "Device:C_Small")
-		(at 114.3 147.32 0)
+		(at 120.65 147.32 0)
 		(unit 1)
 		(exclude_from_sim no)
@@
 		(dnp no)
 		(property "Reference" "C3"
-			(at 108.2601 146.3405 0)
+			(at 114.6101 146.3405 0)
 			(effects
 				(font
@@
 		)
 		(property "Value" "0.1uF"
-			(at 106.9968 148.7928 0)
+			(at 113.3468 148.7928 0)
 			(effects
 				(font
@@
 		)
 		(property "Footprint" "Capacitor_SMD:C_0402_1005Metric"
-			(at 114.3 147.32 0)
+			(at 120.65 147.32 0)
 			(effects
 				(font
@@
 		)
 		(property "Datasheet" "~"
-			(at 114.3 147.32 0)
+			(at 120.65 147.32 0)
 			(effects
 				(font
@@
 		)
 		(property "Description" "100nF 16V X7R ±10% 0402 Multilayer Ceramic Capacitors"
-			(at 114.3 147.32 0)
+			(at 120.65 147.32 0)
 			(effects
 				(font
@@
 		)
 		(property "LCSC" "C1525"
-			(at 114.3 147.32 0)
+			(at 120.65 147.32 0)
 			(effects
 				(font
@@
 		)
 		(property "Link" "https://www.digikey.com/en/products/detail/samsung-electro-mechanics/CL05B104KO5NNNC/3886659"
-			(at 114.3 147.32 0)
+			(at 120.65 147.32 0)
 			(effects
 				(font
@@
 		)
 		(property "Package" "0402 "
-			(at 114.3 147.32 0)
+			(at 120.65 147.32 0)
 			(effects
 				(font
@@
 		)
 		(property "Manu." "Samsung Electro-Mechanics"
-			(at 114.3 147.32 0)
+			(at 120.65 147.32 0)
 			(effects
 				(font
@@
 		)
 		(property "Manu #" "CL05B104KO5NNNC"
-			(at 114.3 147.32 0)
+			(at 120.65 147.32 0)
 			(effects
 				(font
@@
 		)
 		(property "Digikey P/N" ""
-			(at 114.3 147.32 0)
+			(at 120.65 147.32 0)
 			(effects
 				(font
@@
 		)
 		(property "Digikey Page" ""
-			(at 114.3 147.32 0)
+			(at 120.65 147.32 0)
 			(effects
 				(font
@@
 			)
 		)
-		(property "Link" "https://www.mouser.com/ProductDetail/Samsung-Electro-Mechanics/CL31B225KBHNNNE?qs=349EhDEZ59oNolj3jR402w%3D%3D"
+		(property "Link" "https://www.mouser.com/ProductDetail/Samsung-Electro-Mechanics/CL21A225KBQNNNE?qs=xZ%2FP%252Ba9zWqaBMj9IHA8rdw%3D%3D"
 			(at 50.8 81.28 0)
 			(effects
@@
 			)
 		)
-		(property "Manu #" "CL31B225KBHNNNE"
+		(property "Manu #" "CL21A225KBQNNNE"
 			(at 50.8 81.28 0)
 			(effects
@@
 			)
 		)
-		(property "LCSC" "C50254"
-			(at 50.8 81.28 0)
-			(effects
-				(font
-					(size 1.27 1.27)
-				)
-				(hide yes)
-			)
-		)
-		(property "Digikey P/N" ""
-			(at 50.8 81.28 0)
-			(effects
-				(font
-					(size 1.27 1.27)
-				)
-				(hide yes)
-			)
-		)
-		(property "Digikey Page" ""
+		(property "LCSC" "C377773"
 			(at 50.8 81.28 0)
 			(effects
@@
 	(symbol
 		(lib_id "power:+5V")
-		(at 114.3 144.78 0)
+		(at 120.65 144.78 0)
 		(unit 1)
 		(exclude_from_sim no)
@@
 		(dnp no)
 		(property "Reference" "#PWR05"
-			(at 114.3 148.59 0)
+			(at 120.65 148.59 0)
 			(effects
 				(font
@@
 		)
 		(property "Value" "+5V"
-			(at 114.046 140.716 0)
+			(at 120.396 140.716 0)
 			(effects
 				(font
@@
 		)
 		(property "Footprint" ""
-			(at 114.3 144.78 0)
+			(at 120.65 144.78 0)
 			(effects
 				(font
@@
 		)
 		(property "Datasheet" ""
-			(at 114.3 144.78 0)
+			(at 120.65 144.78 0)
 			(effects
 				(font
@@
 		)
 		(property "Description" "Power symbol creates a global label with name \"+5V\""
-			(at 114.3 144.78 0)
+			(at 120.65 144.78 0)
 			(effects
 				(font
@@
 			)
 		)
-		(property "LCSC" "-"
-			(at 66.04 76.2 0)
-			(effects
-				(font
-					(size 1.27 1.27)
-				)
-				(hide yes)
-			)
-		)
-		(property "Digikey P/N" ""
-			(at 66.04 76.2 0)
-			(effects
-				(font
-					(size 1.27 1.27)
-				)
-				(hide yes)
-			)
-		)
-		(property "Digikey Page" ""
+		(property "LCSC" "C22371890"
 			(at 66.04 76.2 0)
 			(effects
@@
 			)
 		)
-		(property "LCSC" "-"
+		(property "LCSC" "C30734"
 			(at 344.17 46.99 0)
 			(effects
@@
 			)
 		)
-		(property "Manu #" " 0402WGF1000TCE"
+		(property "Manu #" "0402WGF1000TCE"
 			(at 85.09 161.29 0)
 			(effects
@@
 			)
 		)
-		(property "Digikey P/N" ""
-			(at 85.09 161.29 90)
-			(effects
-				(font
-					(size 1.27 1.27)
-				)
-				(hide yes)
-			)
-		)
-		(property "Digikey Page" ""
-			(at 85.09 161.29 90)
-			(effects
-				(font
-					(size 1.27 1.27)
-				)
-				(hide yes)
-			)
-		)
 		(pin "2"
 		)
@@
 			)
 		)
-		(property "Digikey P/N" ""
-			(at 344.17 110.49 0)
-			(effects
-				(font
-					(size 1.27 1.27)
-				)
-				(hide yes)
-			)
-		)
-		(property "Digikey Page" ""
-			(at 344.17 110.49 0)
-			(effects
-				(font
-					(size 1.27 1.27)
-				)
-				(hide yes)
-			)
-		)
 		(property "Package" "THT,p=2.54mm"
 			(at 344.17 110.49 0)
@@
 			)
 		)
-		(property "LCSC" "-"
+		(property "LCSC" "C30734"
 			(at 344.17 110.49 0)
 			(effects
@@
 			)
 		)
-		(property "LCSC" "-"
+		(property "LCSC" "C151075"
 			(at 52.07 31.75 90)
 			(effects
@@
 			)
 		)
-		(property "Digikey P/N" ""
-			(at 52.07 31.75 90)
-			(effects
-				(font
-					(size 1.27 1.27)
-				)
-				(hide yes)
-			)
-		)
-		(property "Digikey Page" ""
-			(at 52.07 31.75 90)
-			(effects
-				(font
-					(size 1.27 1.27)
-				)
-				(hide yes)
-			)
-		)
 		(pin "1"
 		)
@@
 			)
 		)
-		(property "LCSC" "-"
+		(property "LCSC" "C89123"
 			(at 21.59 31.75 0)
 			(effects

Commit message: PCB Wrap up
Other:
- company: Meow Wolf -> Daniel Bornhorst
- title: (none) -> Jaquard Machine Driver
Changed lines of the file:
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@@
 	(paper "USLedger")
 	(title_block
-		(rev "v.01")
-		(company "Meow Wolf")
-		(comment 1 "Daniel Bornhorst")
+		(title "Jaquard Machine Driver")
+		(date "2026-09-15")
+		(rev "v1.0")
+		(company "Daniel Bornhorst")
+		(comment 1 "dbornhorst@gmail.com")
 	)
 	(rectangle
